File: Hardware/v3_6_kicad8/odrive.kicad_sch (KiCad schematic)
At the start: 73 parts, among them J3 Leftheader, J4 Rightheader, J9 1868076, U1 SN65HVD232D, U3 AZ1117EH, U8 LP5907

Commit message: update DCBUS voltage divider for 48/56V
Other:
- note added: "56V , R6 改為18K"
Changed lines of the file:
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@@
+		)
+	)
+	(text "56V , R6 改為18K\n"
+		(exclude_from_sim no)
+		(at 362.712 40.894 0)
+		(effects
+			(font
+				(size 1.27 1.27)
+			)
 		)
 	)
